File: AmplifierBoard/AmplifierBoard.kicad_pcb (KiCad board)
At the start: 2 copper layers, 210 x 104 mm, 243 parts, among them J1 12-20V, J2 Digital, J3 AUX1, J4 AUX2, J5 CHANNEL A, J6 CHANNEL B, J7 Frontpanel, J8 ICSP, J9 Serial Debug, U1 TPA3251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

Commit message: firmware revision for real hardware
Parts:
- R7: value 22k -> 27k

Commit message: updated schematic of amplifier board
Parts:
- removed R53, R54: 10k, Resistor_SMD:R_0603_1608Metric_Pad0.98x0.95mm_HandSolder
- added C101: 10µF, Capacitor_SMD:C_0805_2012Metric_Pad1.18x1.45mm_HandSolder, F.Cu at (151.5, 135.5)
- added C102: 10µF, Capacitor_SMD:C_0805_2012Metric_Pad1.18x1.45mm_HandSolder, F.Cu at (142.0, 135.5)
- R42, R45: value 10k -> 0
- R43, R46: value 0 -> 10k
