File: AmplifierBoard/AmplifierBoard.kicad_sch (KiCad schematic)
At the start: 59 parts, among them J1 12-20V, J2 Digital, J3 AUX1, J4 AUX2, J5 CHANNEL A, J6 CHANNEL B, U10 LM1117MP-3.3, U12 PT2258, U14 L7809, U15 LM833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

Commit message: updated schematic of amplifier board
Parts:
- removed R53, R54: 10k, Resistor_SMD:R_0603_1608Metric_Pad0.98x0.95mm_HandSolder, symbol Device:R_Small
- added C101, C102: 10µF, Capacitor_SMD:C_0805_2012Metric_Pad1.18x1.45mm_HandSolder, symbol Device:C_Small
Connections:
- net at R48.2, R50.2, R52.2: now also C102.1
- net at RV2.3, U15.6 (-): now also C102.2
- net at R47.2, R49.2, R51.2: now also C101.1
- net at RV1.3, U15.2 (-): now also C101.2
Changed lines of the file:
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@@
-    )
-  )
-  (symbol (lib_id "Device:R_Small") (at 146.05 152.4 90) (unit 1)
-    (in_bom yes) (on_board yes) (dnp no)
-    (property "Reference" "R54" (at 146.05 150.495 90)
-      (effects (font (size 1.27 1.27)))
-    )
-    (property "Value" "10k" (at 146.05 154.305 90)
-      (effects (font (size 1.27 1.27)))
-    )
-    (property "Footprint" "Resistor_SMD:R_0603_1608Metric_Pad0.98x0.95mm_HandSolder" (at 146.05 152.4 0)
-      (effects (font (size 1.27 1.27)) hide)
-    )
-    (property "Datasheet" "~" (at 146.05 152.4 0)
-      (effects (font (size 1.27 1.27)) hide)
-    )
-    (property "LCSC" "C25804" (at 146.05 150.495 0)
-      (effects (font (size 1.27 1.27)) hide)
-    )
-    (pin "1")
-    (pin "2")
-    (instances
-      (project "AmplifierBoard"
-        (path "/78e63f42-f631-42b6-a0d4-478b86bd13ea"
-          (reference "R54") (unit 1)
-        )
-      )
     )
   )
@@
         (path "/78e63f42-f631-42b6-a0d4-478b86bd13ea"
           (reference "#PWR055") (unit 1)
+        )
+      )
+    )
+  )
+  (symbol (lib_id "Device:C_Small") (at 146.05 152.4 90) (unit 1)
+    (in_bom yes) (on_board yes) (dnp no)
+    (property "Reference" "C102" (at 146.05 155.194 90)
+      (effects (font (size 1.27 1.27)))
+    )
+    (property "Value" "10µF" (at 146.05 157.734 90)
+      (effects (font (size 1.27 1.27)))
+    )
+    (property "Footprint" "Capacitor_SMD:C_0805_2012Metric_Pad1.18x1.45mm_HandSolder" (at 146.05 152.4 0)
+      (effects (font (size 1.27 1.27)) hide)
+    )
+    (property "Datasheet" "~" (at 146.05 152.4 0)
+      (effects (font (size 1.27 1.27)) hide)
+    )
+    (property "LCSC" "C107114" (at 144.7863 149.86 0)
+      (effects (font (size 1.27 1.27)) hide)
+    )
+    (pin "1")
+    (pin "2")
+    (instances
+      (project "AmplifierBoard"
+        (path "/78e63f42-f631-42b6-a0d4-478b86bd13ea"
+          (reference "C102") (unit 1)
         )
       )
@@
     )
   )
+  (symbol (lib_id "Device:C_Small") (at 144.145 133.985 90) (unit 1)
+    (in_bom yes) (on_board yes) (dnp no) (fields_autoplaced)
+    (property "Reference" "C101" (at 144.1513 127 90)
+      (effects (font (size 1.27 1.27)))
+    )
+    (property "Value" "10µF" (at 144.1513 129.54 90)
+      (effects (font (size 1.27 1.27)))
+    )
+    (property "Footprint" "Capacitor_SMD:C_0805_2012Metric_Pad1.18x1.45mm_HandSolder" (at 144.145 133.985 0)
+      (effects (font (size 1.27 1.27)) hide)
+    )
+    (property "Datasheet" "~" (at 144.145 133.985 0)
+      (effects (font (size 1.27 1.27)) hide)
+    )
+    (property "LCSC" "C107114" (at 142.8813 131.445 0)
+      (effects (font (size 1.27 1.27)) hide)
+    )
+    (pin "1")
+    (pin "2")
+    (instances
+      (project "AmplifierBoard"
+        (path "/78e63f42-f631-42b6-a0d4-478b86bd13ea"
+          (reference "C101") (unit 1)
+        )
+      )
+    )
+  )
   (symbol (lib_id "Device:L_Small") (at 214.63 31.75 0) (unit 1)
     (in_bom yes) (on_board yes) (dnp no)
@@
         )
       )
-    )
-  )
-  (symbol (lib_id "Device:R_Small") (at 144.145 133.985 90) (unit 1)
-    (in_bom yes) (on_board yes) (dnp no)
-    (property "Reference" "R53" (at 144.145 132.08 90)
-      (effects (font (size 1.27 1.27)))
-    )
-    (property "Value" "10k" (at 144.145 135.89 90)
-      (effects (font (size 1.27 1.27)))
-    )
-    (property "Footprint" "Resistor_SMD:R_0603_1608Metric_Pad0.98x0.95mm_HandSolder" (at 144.145 133.985 0)
-      (effects (font (size 1.27 1.27)) hide)
-    )
-    (property "Datasheet" "~" (at 144.145 133.985 0)
-      (effects (font (size 1.27 1.27)) hide)
-    )
-    (property "LCSC" "C25804" (at 144.145 132.08 0)
-      (effects (font (size 1.27 1.27)) hide)
-    )
-    (pin "1")
-    (pin "2")
-    (instances
-      (project "AmplifierBoard"
-        (path "/78e63f42-f631-42b6-a0d4-478b86bd13ea"
-          (reference "R53") (unit 1)
-        )
-      )

Commit message: update pcb version
Parts:
- renumbered C56 to C84, C58 to C85, L8 to L14, L7 to L15
