File: AmplifierBoard/AnalogBuffers.kicad_sch (KiCad schematic)
At the start: 38 parts, among them U11 LM833

Commit message: update pcb version
Parts:
- renumbered C56 to C66, C58 to C67, C56 to C68, C58 to C69, C64 to C70, C65 to C71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
