File: AmplifierBoard/AudioDetect.kicad_sch (KiCad schematic)
At the start: 16 parts, among them U16 LM358, U17 74HC14

Commit message: updated schematic of amplifier board
Parts:
- R42, R45: value 10k -> 0
- R43, R46: value 0 -> 10k
Changed lines of the file:
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@@
       (effects (font (size 1.27 1.27)))
     )
-    (property "Value" "10k" (at 93.98 78.74 90)
+    (property "Value" "0" (at 93.98 78.74 90)
       (effects (font (size 1.27 1.27)))
     )
@@
       (effects (font (size 1.27 1.27)))
     )
-    (property "Value" "10k" (at 93.98 46.99 90)
+    (property "Value" "0" (at 93.98 46.99 90)
       (effects (font (size 1.27 1.27)))
     )
@@
       (effects (font (size 1.27 1.27)))
     )
-    (property "Value" "0" (at 114.3 38.1 90)
+    (property "Value" "10k" (at 114.3 38.1 90)
       (effects (font (size 1.27 1.27)))
     )
@@
       (effects (font (size 1.27 1.27)))
     )
-    (property "Value" "0" (at 114.3 69.85 90)
-      (effects (font (size 1.27 1.27)))
-    )
+    (property "Value" "10k" (at 114.3 69.85 90)
+      (effects (font (size 1.27 1.27)))
+    )

Commit message: update pcb version
Parts:
- renumbered C56 to C80, C58 to C81, L8 to L12, L7 to L13
