File: AmplifierBoard/MCU.kicad_sch (KiCad schematic)
At the start: 15 parts, among them J7 Frontpanel, J8 ICSP, J9 Serial Debug, U18 ATmega328PB-A

Commit message: update pcb version
Parts:
- renumbered C56 to C88, C56 to C89, C56 to C91, C56 to C92, L8 to L16, L7 to L18
