File: AmplifierBoard/PowerAmp.kicad_sch (KiCad schematic)
At the start: 49 parts

Commit message: update pcb version
Parts:
- gave numbers to parts that had none: 35
- renumbered L8 to L17, L8 to L19
