File: AmplifierBoard/TosLink.kicad_sch (KiCad schematic)
At the start: 52 parts, among them U5 PCM1793, U6 WM8804, U7 LM833, U8 MIC811TUY, Y1 12MHz

Commit message: update pcb version
Parts:
- renumbered C65 to C100, C65 to C99, R30 to R57, R30 to R58
